File: cad/1_1/1_1.kicad_pcb (KiCad board)
At the start: 2 copper layers, 80 x 50 mm, 14 parts, among them J1 Conn_01x04_Pin, U1 ATtiny1616-M

Commit message: I love Japan
Parts:
- added G***: LOGO, LOGO, B.Cu at (90.0, 75.0)
Other:
- board text added: "Hinomaru SiliCa v1.1.2h"
- board text removed: "SiliCa v1.1.2"
Changed lines of the file:
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@@
 		)
+	)
+	(footprint "LOGO"
+		(layer "B.Cu")
+		(at 90 75 180)
+		(property "Reference" "G***"
+			(at 0 0 0)
+			(layer "B.SilkS")
+			(hide yes)
+			(effects
+				(font
+					(size 1.5 1.5)
+					(thickness 0.3)
+				)
+				(justify mirror)
+			)
+		)
+		(property "Value" "LOGO"
+			(at 0.75 0 0)
+			(layer "B.SilkS")
+			(hide yes)
+			(effects
+				(font
+					(size 1.5 1.5)
+					(thickness 0.3)
+				)
+				(justify mirror)
+			)
+		)
+		(property "Datasheet" ""
+			(at 0 0 0)
+			(layer "B.Fab")
+			(hide yes)
+			(effects
+				(font
+					(size 1.27 1.27)
+					(thickness 0.15)
+				)
+				(justify mirror)
+			)
+		)
+		(property "Description" ""
+			(at 0 0 0)
+			(layer "B.Fab")
+			(hide yes)
+			(effects
+				(font
+					(size 1.27 1.27)
+					(thickness 0.15)
+				)
+				(justify mirror)
+			)
+		)
+		(attr board_only exclude_from_pos_files exclude_from_bom)
+		(fp_poly
+			(pts
+				(xy 40.035026 0.000001) (xy 40.035026 -26.690017) (xy 0 -26.690017) (xy -40.035026 -26.690017) (xy -40.035026 0.000001)
+				(xy -15.988553 0.000001) (xy -15.97451 -0.791334) (xy -15.93029 -1.524794) (xy -15.852758 -2.22726)
+				(xy -15.738778 -2.925615) (xy -15.585212 -3.64674) (xy -15.542269 -3.825568) (xy -15.220866 -4.95324)
+				(xy -14.818592 -6.048519) (xy -14.338793 -7.107465) (xy -13.784815 -8.126138) (xy -13.160003 -9.100599)
+				(xy -12.467703 -10.02691) (xy -11.71126 -10.901129) (xy -10.894019 -11.719318) (xy -10.019327 -12.477538)
+				(xy -9.090528 -13.171849) (xy -8.110967 -13.798311) (xy -7.083991 -14.352986) (xy -6.294396 -14.715369)
+				(xy -5.601053 -14.994965) (xy -4.925091 -15.234007) (xy -4.250075 -15.436366) (xy -3.559567 -15.605909)
+				(xy -2.837129 -15.746507) (xy -2.066326 -15.86203) (xy -1.230719 -15.956346) (xy -0.889667 -15.9877)
+				(xy -0.715402 -15.996274) (xy -0.470274 -15.999298) (xy -0.172179 -15.99733) (xy 0.16099 -15.990929)
+				(xy 0.511338 -15.980652) (xy 0.86097 -15.967057) (xy 1.191992 -15.950704) (xy 1.48651 -15.932149)
+				(xy 1.726628 -15.911951) (xy 1.801576 -15.90376) (xy 3.002269 -15.718259) (xy 4.164314 -15.453057)
+				(xy 5.290454 -15.107208) (xy 6.383428 -14.679765) (xy 7.445978 -14.169781) (xy 8.407355 -13.621753)
+				(xy 9.309068 -13.019048) (xy 10.183138 -12.339481) (xy 11.019142 -11.593474) (xy 11.806658 -10.791451)
+				(xy 12.535263 -9.943834) (xy 13.194536 -9.061044) (xy 13.621754 -8.407355) (xy 14.16928 -7.441478)
+				(xy 14.652642 -6.432592) (xy 15.06688 -5.393929) (xy 15.407037 -4.338723) (xy 15.668152 -3.280207)
+				(xy 15.78874 -2.624517) (xy 15.856333 -2.17738) (xy 15.907555 -1.779328) (xy 15.944383 -1.404406)
+				(xy 15.968792 -1.026657) (xy 15.982758 -0.620128) (xy 15.988257 -0.158863) (xy 15.988552 0.000001)
+				(xy 15.974509 0.791336) (xy 15.93029 1.524796) (xy 15.852758 2.227262) (xy 15.738777 2.925617) (xy 15.585212 3.646742)
+				(xy 15.542269 3.82557) (xy 15.219582 4.958231) (xy 14.815804 6.057921) (xy 14.333878 7.120885) (xy 13.776745 8.143368)
+				(xy 13.147346 9.121618) (xy 12.448625 10.051879) (xy 11.683522 10.930398) (xy 10.85498 11.753421)
+				(xy 9.96594 12.517192) (xy 9.019344 13.217959) (xy 8.018134 13.851966) (xy 7.428721 14.179614) (xy 6.396657 14.676124)
+				(xy 5.320865 15.096494) (xy 4.200295 15.441037) (xy 3.033894 15.710069) (xy 1.820613 15.903905)
+				(xy 1.579159 15.93289) (xy 1.333197 15.953663) (xy 1.017626 15.969397) (xy 0.651662 15.980092) (xy 0.254519 15.985748)
+				(xy -0.154587 15.986366) (xy -0.556441 15.981945) (xy -0.931827 15.972485) (xy -1.261531 15.957987)
+				(xy -1.526337 15.938449) (xy -1.57916 15.93289) (xy -2.636967 15.784736) (xy -3.63735 15.585676)
+				(xy -4.598984 15.330887) (xy -5.540545 15.015547) (xy -6.294396 14.715371) (xy -7.351155 14.217622)
+				(xy -8.366335 13.643304) (xy -9.335799 12.996553) (xy -10.255415 12.281502) (xy -11.121048 11.502286)
+				(xy -11.928564 10.66304) (xy -12.673828 9.767896) (xy -13.352705 8.82099) (xy -13.961063 7.826456)
+				(xy -14.494766 6.788428) (xy -14.71537 6.294397) (xy -15.12355 5.244151) (xy -15.449906 4.199113)
+				(xy -15.696971 3.146762) (xy -15.867276 2.074578) (xy -15.963354 0.970039) (xy -15.988553 0.000001)
+				(xy -40.035026 0.000001) (xy -40.035026 26.690018) (xy 0 26.690018) (xy 40.035026 26.690018)
+			)
+			(stroke
+				(width 0)
+				(type solid)
+			)
+			(fill yes)
+			(layer "B.SilkS")
+		)
+		(embedded_fonts no)
 	)
 	(gr_rect
@@
 		(locked yes)
 		(layer "Edge.Cuts")
+	)
+	(gr_rect
+		(start 82.5 72.5)
+		(end 97.5 77.5)
+		(stroke
+			(width 0.15)
+			(type default)
+		)
+		(fill no)
+		(layer "User.1")
 	)
 	(gr_line
@@
 		(layer "User.1")
 	)
-	(gr_rect
-		(start 82.5 72.5)
-		(end 97.5 77.5)
-		(stroke
-			(width 0.15)
-			(type default)
+	(gr_text "UPDI"
+		(at 118 72 0)
+		(layer "F.SilkS")
+		(effects
+			(font
+				(size 1 1)
+				(thickness 0.15)
+			)
+			(justify left bottom)
 		)
-		(fill no)
-		(layer "User.1")
+	)
+	(gr_text "GND"
+		(at 118.5 74.5 0)
+		(layer "F.SilkS")
+		(effects
+			(font
+				(size 1 1)
+				(thickness 0.15)
+			)
+			(justify left bottom)
+		)
 	)
 	(gr_text "VCC"
@@
 		)
 	)
-	(gr_text "GND"
-		(at 118.5 74.5 0)
-		(layer "F.SilkS")
-		(effects
-			(font
-				(size 1 1)
-				(thickness 0.15)
-			)
-			(justify left bottom)
-		)
-	)
-	(gr_text "SiliCa v1.1.2"
-		(at 115.5 93.5 0)
+	(gr_text "Hinomaru SiliCa v1.1.2h"
+		(at 107 93.5 0)
 		(layer "F.SilkS")
 		(effects
@@
 		)
 	)
-	(gr_text "UPDI"
-		(at 118 72 0)
-		(layer "F.SilkS")
-		(effects
-			(font
-				(size 1 1)
-				(thickness 0.15)
-			)
-			(justify left bottom)
-		)
-	)
